File: DazzerBlue-proj/DazzerBlue-proj.kicad_pcb (KiCad board)
At the start: 2 copper layers, 32 x 62.5 mm, 11 parts

Commit message: Added self-made V101S model to PCB
Other:
- outline, holes or cut-outs redrawn
- board text added: "V101S DHE537"
Changed lines of the file:
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@@
 		)
 		(embedded_fonts no)
+		(model "${KIPRJMOD}/models_external/V101S_model_C0m3b4ck.step"
+			(offset
+				(xyz 11.25 11 0)
+			)
+			(scale
+				(xyz 1 1 1)
+			)
+			(rotate
+				(xyz -0 -0 90)
+			)
+		)
 	)
 	(footprint "LED_THT:LED_D3.0mm_Horizontal_O1.27mm_Z2.0mm_Clear"
@@
 	)
 	(gr_rect
+		(start 167 69)
+		(end 176.5 96)
+		(stroke
+			(width 0.05)
+			(type default)
+		)
+		(fill no)
+		(layer "Edge.Cuts")
+	)
+	(gr_rect
 		(start 167.5 47.5)
 		(end 174.5 66)
@@
 		(layer "Edge.Cuts")
 	)
+	(gr_text "V101S	\nDHE537"
+		(at 169 78.5 0)
+		(layer "F.SilkS")
+		(effects
+			(font
+				(size 1 1)
+				(thickness 0.1)
+			)
+			(justify left bottom)
+		)
+	)
 	(embedded_fonts no)

Commit message: Finished project, updated README
Parts:
- added ?: , , F.Cu at (183.5, 103.0)
- added ?: , , F.Cu at (185.0, 61.5)
- added ?: , , F.Cu at (159.0, 61.5)
- added ?: , , F.Cu at (158.0, 102.5)
- +: footprint LED_THT:LED_D3.0mm_Horizontal_O1.27mm_Z2.0mm_Clear -> NoCourtyard:NoCourtyard_LED_D3.0mm_Horizontal_O1.27mm_Z2.0mm_Clear
- C1, C2: footprint SmallCapacitor:SmallCapacitor -> SmallCapacitor2:SmallCapacitor2
- R4: renamed from R2; footprint Resistor_THT:R_Axial_DIN0204_L3.6mm_D1.6mm_P5.08mm_Vertical -> NoCourtyard:NoCourtyard_R_Axial_DIN0204_L3.6mm_D1.6mm_P5.08mm_Vertical
- R5: renamed from R1; footprint Resistor_THT:R_Axial_DIN0204_L3.6mm_D1.6mm_P5.08mm_Vertical -> NoCourtyard:NoCourtyard_R_Axial_DIN0204_L3.6mm_D1.6mm_P5.08mm_Vertical
- moved U1 14.6 mm to (164.5, 80.0), turned to -90 degrees
- moved CON1 11.2 mm to (186.5, 85.5), turned to 180 degrees
- moved R4 4.99 mm to (186.0, 94.5), turned to 180 degrees
- moved R5 4.98 mm to (186.0, 91.5), turned to 180 degrees
- moved C2 3.04 mm to (181.5, 73.0)
- moved C1 0.71 mm to (184.5, 70.0)
- moved SWL 0.14 mm to (155.5, 55.0)
Connections:
- C1 pad 1: Net-(CON1-VCC) -> Net-(CON1-GND)
- C2 pad 1: Net-(CON1-VCC) -> Net-(CON1-GND)
- C2 pad 2: Net-(CON1-GND) -> Net-(C2-Pad2)
- R4 pad 1: Net-(D1-A) -> Net-(D1-K)
- R5 pad 1: Net-(D1-A) -> Net-(D1-K)
- U1 pad 2: Net-(CON1-GND) -> Net-(C2-Pad2)
- U1 pad 5: Net-(D1-K) -> Net-(D1-A)
- U1 pad 6: Net-(D1-A) -> Net-(D1-K)
- U1 pad 8: Net-(ENC1-A) -> Net-(ENC1-B)
- U1 pad 9: Net-(ENC1-B) -> Net-(ENC1-A)
Routing:
- net Net-(CON1-VCC): track 0.00 -> 220.6 mm
- net Net-(CON1-GND): track 0.00 -> 122.9 mm
- net Net-(SWR1-NO): track 0.00 -> 97.6 mm
- net Net-(SWM1-NO): track 0.00 -> 86.2 mm
- net Net-(SWL1-NO): track 0.00 -> 36.0 mm
- net Net-(D1-K): track 0.00 -> 34.8 mm
- net Net-(ENC1-B): track 0.00 -> 28.3 mm
- net Net-(ENC1-A): track 0.00 -> 27.9 mm
- net Net-(D1-A): track 0.00 -> 20.2 mm
- net Net-(CON1-D2): track 0.00 -> 5.91 mm
- net Net-(CON1-D1): track 0.00 -> 5.91 mm
- added copper zone on B.Cu, net (none)
- added copper zone on B.Cu, net Net-(CON1-GND)
Other:
- board size 32 x 62.5 mm -> 32 x 62 mm
- board text added: "2H-0001"
- board text added: "FRS-MS-310 V1.2 2018.09.25"
- board text added: "IC1"
- board text removed: "V101S DHE537"
