File: DazzerBlue-proj/DazzerBlue-proj.kicad_sch (KiCad schematic)
At the start: 11 parts

Commit message: Finished project, updated README
Parts:
- C1, C2: footprint IllinoisCapacitor_r3mm_h8mm:IllinoisCapacitor_r3mm_h8mm -> SmallCapacitor2:SmallCapacitor2
Connections:
- net at C1.1, CON1.3 (VCC), ENC1.3 (C)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: no longer C2.1
- net at C1.2, CON1.4 (GND), SWL1.1 (C)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: now also C2.1; no longer C2.2, U1.2 (GND)
- net at U1.5 (LED_GND): now also D1.2 (A); no longer D1.1 (K)
- net at R1.1, R2.1, U1.6 (LED_VCC): now also D1.1 (K); no longer D1.2 (A)
- net at U1.8 (ENC1): now also ENC1.2 (B); no longer ENC1.1 (A)
- net at U1.9 (ENC2): now also ENC1.1 (A); no longer ENC1.2 (B)
- new net: C2.2, U1.2 (GND)
Other:
- moved on the sheet: C2, CON1, D1, ENC1, R1, R2
